File: lowimp121.kicad_pcb (KiCad board)
At the start: 2 copper layers, 69.5 x 59 mm, 2 parts, among them M1 Module-vr-max9924-0.1, M2 Module-mega-mcu144-0.6

Commit message: test2
Parts:
- added G***: LOGO, hellen-one-common:LOGO, B.Cu at (267.5, 111.0)
- added G4: DISCLAIMER, rusefi_lib:Off_Road_Disclaimer, B.Cu at (190.0, 106.9)
- added M3: Module-input-0.1, INPUT:input, F.Cu at (211.3, 174.5)
- added M4: Module-mcu-0.7, MCU:mcu, F.Cu at (211.3, 158.5)
- added M5: Module-power_12and5V-0.1, POWER:power_12and5V, F.Cu at (259.1, 141.9)
- added M6: Module-stlink-0.1, ST_LINK:stlink, F.Cu at (243.7, 185.7)
- added M7: Module-wbo-0.5, WBO:wbo, F.Cu at (243.7, 173.8)
- added P2: 368255-2, kicad6-libraries:TE_368255-2, F.Cu at (262.4, 198.4)
- M1: footprint 0.3:vr-max9924 -> VR_9924:vr-max9924
- M2: value Module-mega-mcu144-0.6 -> Module-ign8-0.2; footprint 0.6:mega-mcu144 -> IGN:ign8
- moved M2 162.2 mm to (259.1, 157.0)
- moved M1 135.1 mm to (211.3, 185.6)
Connections:
- M1 pad E4: Net-(M1-V5_IN) -> unconnected-(M1-V5_IN-PadE4)
- M1 pad G: Net-(M1-GND) -> unconnected-(M1-GND-PadG)
- M1 pad W1: Net-(M1-VR-/HALL) -> unconnected-(M1-VR-/HALL-PadW1)
- M1 pad W2: Net-(M1-VR+) -> unconnected-(M1-VR+-PadW2)
Routing:
- net (no net): vias 0 -> 31
- added copper zone on B.Cu, net (none)
- added copper zone on F.Cu, net (none)
- added copper zone on In1.Cu, net (none)
Other:
- board size 69.5 x 59 mm -> 164 x 118 mm
- copper layers 2 -> 4
