File: lowimp121.kicad_sch (KiCad schematic)
At the start: 2 parts, among them M1 Module-vr-max9924-0.1, M2 Module-mega-mcu144-0.6

Commit message: test2
Parts:
- removed M2: Module-mega-mcu144-0.6, 0.6:mega-mcu144, symbol mega-mcu144:Module-mega-mcu144-0.6
- added M2: Module-ign8-0.2, IGN:ign8, symbol ign8:Module-ign8-0.2
- added M3: Module-input-0.1, INPUT:input, symbol input:Module-input-0.1
- added M4: Module-mcu-0.7, MCU:mcu, symbol mcu:Module-mcu-0.7
- added M5: Module-power_12and5V-0.1, POWER:power_12and5V, symbol power_12and5V:Module-power_12and5V-0.1
- added M6: Module-stlink-0.1, ST_LINK:stlink, symbol stlink:Module-stlink-0.1
- added M7: Module-wbo-0.5, WBO:wbo, symbol wbo:Module-wbo-0.5
- added P2: 368255-2, kicad6-libraries:TE_368255-2, symbol TE_368255-2:368255-2
- M1: footprint 0.3:vr-max9924 -> VR_9924:vr-max9924
Other:
- company: (none) -> andreika @ rusEFI.com
- title: (none) -> Hellen121vag
